Commit message: double limit commented out

File: suturo_resources/urdf/urdf_components/suturo_kitchen.urdf.xacro (robot description, xacro)
@@ -850,5 +850,5 @@
     <axis xyz="1. 0. 0.0"/>
     <limit effort="300" lower="0" upper="0.48" velocity="10"/>
-        <limit effort="300" lower="0" upper="0" velocity="10"/>
+	<!--<limit effort="300" lower="0" upper="0" velocity="10"/>-->
   </joint>
   <joint name="oven_area_area_left_drawer_handle_joint" type="fixed">

Commit message: changed iai_fridge_door_joint from revolute to fixed for testing

File: suturo_resources/urdf/urdf_components/suturo_kitchen.urdf.xacro (robot description, xacro)
@@ -1912,5 +1912,5 @@
     <child link="iai_fridge_main"/>
   </joint>
-  <joint name="iai_fridge_door_joint" type="revolute">
+  <joint name="iai_fridge_door_joint" type="fixed">
     <origin rpy="0 0 0" xyz="0.29 0.3 0.245"/>
     <parent link="iai_fridge_main"/>

Commit message: changed iai_fridge_door_joint back to  revolute

File: suturo_resources/urdf/urdf_components/suturo_kitchen.urdf.xacro (robot description, xacro)
@@ -1912,5 +1912,5 @@
     <child link="iai_fridge_main"/>
   </joint>
-  <joint name="iai_fridge_door_joint" type="fixed">
+  <joint name="iai_fridge_door_joint" type="revolute">
     <origin rpy="0 0 0" xyz="0.29 0.3 0.245"/>
     <parent link="iai_fridge_main"/>
